File: hardware/wifi-leds.sch (EAGLE design)
At the start: 30 parts, among them IC2 LDL112D33R, Q2 FQP30N06L, U1 ESP-WROOM-32

Commit message: added logo
Parts:
- added U$5: CMD_C0DE_LOGOCMD_CODE_LOGO_TOP_COPPER, logos:CMD_C0DE_LOGOCMD_CODE_LOGO_TOP_COPPER
Changed lines of the file:
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@@
 <part name="LEDS" library="connector" deviceset="M04" device="POLAR"/>
 <part name="Q2" library="transitors" deviceset="FQP30N06L" device=""/>
+<part name="U$5" library="logos" deviceset="CMD_C0DE_LOGO" device="CMD_CODE_LOGO_TOP_COPPER"/>
 </parts>
 <sheets>
@@
 </nets>
 </sheet>
+<sheet>
+<plain>
+</plain>
+<instances>
+<instance part="U$5" gate="G$1" x="48.26" y="53.34" smashed="yes"/>
+</instances>
+<busses>
+</busses>
+<nets>
+</nets>
+</sheet>
