File: hardware/wifi-leds2.brd (EAGLE design)
At the start: 83 x 59 mm, 50 parts, among them IC2 LDL112D33R, J1 USB-TYPE-B, J3 Battery, Q2 FQP30N06L, U1 ESP-WROOM-32, U2 MCP9700T-E/TT, Y1 ABM7-12.000MHZ-D2Y-T

Commit message: updated gnd
Parts:
- moved U$5 31.4 mm to (75.7, 25.1), flipped to the bottom
Routing:
- net GND: track 11.0 -> 15.2 mm
